Commit message: bicycle control seems to work!

File: src/pca9685_ros2_control/rc_hardware_control/description/description.urdf.xacro (robot description, xacro)
@@ -1,4 +1,11 @@
 <?xml version="1.0"?>
 <robot xmlns:xacro="http://www.ros.org/wiki/xacro" name="rc_car">
+  <!-- Dummy root link to handle KDL inertia requirement -->
+  <link name="base_footprint"/>
+  <joint name="base_footprint_joint" type="fixed">
+    <parent link="base_footprint"/>
+    <child link="base_link"/>
+    <origin xyz="0 0 0" rpy="0 0 0"/>
+  </joint>
   <!-- Chassis: AMORIL 1/10 RC Car -->
   <link name="base_link">
@@ -176,4 +183,5 @@
       <state_interface name="position" />
       <param name="channel">0</param>
+      <param name="offset">0.0</param>
       <param name="min_angle">-0.785</param>
       <param name="max_angle">0.785</param>
@@ -187,5 +195,4 @@
       <state_interface name="position" />
       <param name="channel">1</param>
-      <command_interface name="velocity" />
       <param name="min_pulse_us">1000</param>
       <param name="neutral_pulse_us">1500</param>
