Commit message: local map!   plan!   follow plan needs work

File: src/RCCar/rc_hardware_control/description/description.urdf.xacro (robot description, xacro)
@@ -132,5 +132,5 @@
     <parent link="base_link"/>
     <child link="camera_link"/>
-    <origin xyz="0.20 0 0.127" rpy="3.14159 0 0"/>
+    <origin xyz="0.20 0 0.127" rpy="0 0 0"/>
   </joint>
   <link name="camera_infra1_optical_frame"/>

Commit message: qk save

File: src/RCCar/rc_hardware_control/description/description.urdf.xacro (robot description, xacro)
@@ -87,5 +87,5 @@
     <parent link="steering_link"/>
     <child link="front_left_wheel"/>
-    <origin xyz="0.145 0.11 0.045" rpy="0 0 0"/>
+    <origin xyz="0 0.11 0.045" rpy="0 0 0"/>
     <axis xyz="0 1 0"/>
   </joint>
@@ -93,5 +93,5 @@
     <parent link="steering_link"/>
     <child link="front_right_wheel"/>
-    <origin xyz="0.145 -0.11 0.045" rpy="0 0 0"/>
+    <origin xyz="0 -0.11 0.045" rpy="0 0 0"/>
     <axis xyz="0 1 0"/>
   </joint>
@@ -99,5 +99,5 @@
     <parent link="traction_link"/>
     <child link="rear_left_wheel"/>
-    <origin xyz="-0.145 0.11 0.045" rpy="0 0 0"/>
+    <origin xyz="0 0.11 0.045" rpy="0 0 0"/>
     <axis xyz="0 1 0"/>
   </joint>
@@ -105,5 +105,5 @@
     <parent link="traction_link"/>
     <child link="rear_right_wheel"/>
-    <origin xyz="-0.145 -0.11 0.045" rpy="0 0 0"/>
+    <origin xyz="0 -0.11 0.045" rpy="0 0 0"/>
     <axis xyz="0 1 0"/>
   </joint>
@@ -119,5 +119,5 @@
     <parent link="base_link"/>
     <child link="steering_link"/>
-    <origin xyz="0 0 0" rpy="0 0 0"/>
+    <origin xyz="0.145 0 0" rpy="0 0 0"/>
     <axis xyz="0 0 1"/>
     <limit lower="-1.57" upper="1.57" effort="1" velocity="1"/>
@@ -126,6 +126,6 @@
     <parent link="base_link"/>
     <child link="traction_link"/>
-    <origin xyz="0 0 0" rpy="0 0 0"/>
-    <axis xyz="0 0 1"/>
+    <origin xyz="-0.145 0 0" rpy="0 0 0"/>
+    <axis xyz="0 1 0"/>
   </joint>
   <joint name="camera_joint" type="fixed">
