Commit message: Make frames and dimensions consistent (#2)
base_footprint is now a true ground frame and base_link the chassis frame
at axle height, joined by the wheel radius. Chassis box, wheels and camera
are shifted so their real-world heights are unchanged; previously base_link
sat on the ground and the chassis was drawn half underground.

All dimensions are xacro properties. Wheel radius 0.049 m (owner-reported
diameter just under 4 in) replaces 0.045 in the URDF and 0.035 in the
steering controller. Steering joint limit now matches the servo range.
Every launch file points visual SLAM and nvblox at base_footprint. The
planner's minimum turning radius carries its derivation and a floor based
on a typical 1/10 lock angle, since the mechanical lock is unmeasured.

Still open on #2: ground clearance is an estimate, and the live transform
checks need the Isaac container.

Co-Authored-By: Claude Fable 5.1 <noreply@anthropic.com>
Claude-Session: https://claude.ai/code/session_015xtnKLNTCcXYNkdv7Yybut

File: src/RCCar/rc_hardware_control/description/description.urdf.xacro (robot description, xacro)
@@ -1,21 +1,51 @@
 <?xml version="1.0"?>
 <robot xmlns:xacro="http://www.ros.org/wiki/xacro" name="rc_car">
-  <!-- Dummy root link to handle KDL inertia requirement -->
+  <!-- ============================================================
+       Physical dimensions. Every frame below is derived from these.
+       wheel_radius: owner reported the wheel diameter as "just under
+       4 inches" (2026-09-12), taken as 0.098 m. Replace with a caliper
+       measurement when one is made. The same value must be written in
+       config/steer_bot_hardware.yaml (front/rear_wheel_radius).
+       ground_clearance: ESTIMATE, not yet measured. It only affects
+       where the chassis box is drawn, not any frame, but the obstacle
+       height band in the nvblox config was chosen relative to it.
+       steer_max_angle: the PCA9685 calibration range, not a measured
+       mechanical lock. See the turning-radius note in
+       config/my_custom_nav2_params.yaml.
+       ============================================================ -->
+  <xacro:property name="wheel_radius"      value="0.049"/>
+  <xacro:property name="wheel_width"       value="0.04"/>
+  <xacro:property name="wheelbase"         value="0.29"/>
+  <xacro:property name="track_width"       value="0.22"/>
+  <xacro:property name="chassis_length"    value="0.44"/>
+  <xacro:property name="chassis_width"     value="0.27"/>
+  <xacro:property name="chassis_height"    value="0.15"/>
+  <xacro:property name="ground_clearance"  value="0.04"/>   <!-- ESTIMATE: measure -->
+  <xacro:property name="camera_height"     value="0.127"/>  <!-- lens centre above ground -->
+  <xacro:property name="camera_forward"    value="0.20"/>   <!-- lens ahead of the axle midpoint -->
+  <xacro:property name="steer_max_angle"   value="0.785"/>  <!-- servo hardware limit, rad -->
+  <!-- Frames:
+       base_footprint  ground-contact frame, z = 0 on the floor, midway between the axles.
+       base_link       chassis frame at axle height, wheel_radius above base_footprint.
+       Nav2, visual SLAM and nvblox all use base_footprint as the robot frame. -->
   <link name="base_footprint"/>
   <joint name="base_footprint_joint" type="fixed">
     <parent link="base_footprint"/>
     <child link="base_link"/>
-    <origin xyz="0 0 0" rpy="0 0 0"/>
-  </joint>
-  <!-- Chassis: AMORIL 1/10 RC Car -->
+    <origin xyz="0 0 ${wheel_radius}" rpy="0 0 0"/>
+  </joint>
+  <!-- Chassis: AMORIL 1/10 RC Car. Box centre sits ground_clearance + chassis_height/2
+       above the floor, expressed relative to base_link at axle height. -->
+  <xacro:property name="chassis_centre_z" value="${ground_clearance + chassis_height/2 - wheel_radius}"/>
   <link name="base_link">
     <inertial>
-      <origin xyz="0 0 0.075"/>
+      <origin xyz="0 0 ${chassis_centre_z}"/>
       <mass value="3.0"/>
       <inertia ixx="0.08" ixy="0.0" ixz="0.0" iyy="0.25" iyz="0.0" izz="0.28"/>
     </inertial>
     <visual>
-      <geometry>
-        <box size="0.44 0.27 0.15"/>
+      <origin xyz="0 0 ${chassis_centre_z}"/>
+      <geometry>
+        <box size="${chassis_length} ${chassis_width} ${chassis_height}"/>
       </geometry>
       <material name="gray">
@@ -24,6 +54,7 @@
     </visual>
     <collision>
-      <geometry>
-        <box size="0.44 0.27 0.15"/>
+      <origin xyz="0 0 ${chassis_centre_z}"/>
+      <geometry>
+        <box size="${chassis_length} ${chassis_width} ${chassis_height}"/>
       </geometry>
     </collision>
@@ -33,5 +64,5 @@
     <visual>
       <geometry>
-        <cylinder length="0.04" radius="0.045"/>
+        <cylinder length="${wheel_width}" radius="${wheel_radius}"/>
       </geometry>
       <material name="black"><color rgba="0.1 0.1 0.1 1"/></material>
@@ -39,5 +70,5 @@
     <collision>
       <geometry>
-        <cylinder length="0.04" radius="0.045"/>
+        <cylinder length="${wheel_width}" radius="${wheel_radius}"/>
       </geometry>
     </collision>
@@ -46,5 +77,5 @@
     <visual>
       <geometry>
-        <cylinder length="0.04" radius="0.045"/>
+        <cylinder length="${wheel_width}" radius="${wheel_radius}"/>
       </geometry>
       <material name="black"/>
@@ -52,5 +83,5 @@
     <collision>
       <geometry>
-        <cylinder length="0.04" radius="0.045"/>
+        <cylinder length="${wheel_width}" radius="${wheel_radius}"/>
       </geometry>
     </collision>
@@ -59,5 +90,5 @@
     <visual>
       <geometry>
-        <cylinder length="0.04" radius="0.045"/>
+        <cylinder length="${wheel_width}" radius="${wheel_radius}"/>
       </geometry>
       <material name="black"/>
@@ -65,5 +96,5 @@
     <collision>
       <geometry>
-        <cylinder length="0.04" radius="0.045"/>
+        <cylinder length="${wheel_width}" radius="${wheel_radius}"/>
       </geometry>
     </collision>
@@ -72,5 +103,5 @@
     <visual>
       <geometry>
-        <cylinder length="0.04" radius="0.045"/>
+        <cylinder length="${wheel_width}" radius="${wheel_radius}"/>
       </geometry>
       <material name="black"/>
@@ -78,14 +109,14 @@
     <collision>
       <geometry>
-        <cylinder length="0.04" radius="0.045"/>
+        <cylinder length="${wheel_width}" radius="${wheel_radius}"/>
       </geometry>
     </collision>
   </link>
   <!-- Wheel joints (front: steerable, rear: fixed) -->
-  <!-- Wheelbase: 0.29m, track width: 0.22m -->
+  <!-- Axles lie in the base_link plane; wheels sit half a track width to each side. -->
   <joint name="front_left_wheel_joint" type="continuous">
     <parent link="steering_link"/>
     <child link="front_left_wheel"/>
-    <origin xyz="0 0.11 0.045" rpy="0 0 0"/>
+    <origin xyz="0 ${track_width/2} 0" rpy="0 0 0"/>
     <axis xyz="0 1 0"/>
   </joint>
@@ -93,5 +124,5 @@
     <parent link="steering_link"/>
     <child link="front_right_wheel"/>
-    <origin xyz="0 -0.11 0.045" rpy="0 0 0"/>
+    <origin xyz="0 ${-track_width/2} 0" rpy="0 0 0"/>
     <axis xyz="0 1 0"/>
   </joint>
@@ -99,5 +130,5 @@
     <parent link="traction_link"/>
     <child link="rear_left_wheel"/>
-    <origin xyz="0 0.11 0.045" rpy="0 0 0"/>
+    <origin xyz="0 ${track_width/2} 0" rpy="0 0 0"/>
     <axis xyz="0 1 0"/>
   </joint>
@@ -105,5 +136,5 @@
     <parent link="traction_link"/>
     <child link="rear_right_wheel"/>
-    <origin xyz="0 -0.11 0.045" rpy="0 0 0"/>
+    <origin xyz="0 ${-track_width/2} 0" rpy="0 0 0"/>
     <axis xyz="0 1 0"/>
   </joint>
@@ -119,12 +150,12 @@
     <parent link="base_link"/>
     <child link="steering_link"/>
-    <origin xyz="0.145 0 0" rpy="0 0 0"/>
+    <origin xyz="${wheelbase/2} 0 0" rpy="0 0 0"/>
     <axis xyz="0 0 1"/>
-    <limit lower="-1.57" upper="1.57" effort="1" velocity="1"/>
+    <limit lower="${-steer_max_angle}" upper="${steer_max_angle}" effort="1" velocity="1"/>
   </joint>
   <joint name="traction_joint" type="continuous">
     <parent link="base_link"/>
     <child link="traction_link"/>
-    <origin xyz="-0.145 0 0" rpy="0 0 0"/>
+    <origin xyz="${-wheelbase/2} 0 0" rpy="0 0 0"/>
     <axis xyz="0 1 0"/>
   </joint>
@@ -132,5 +163,5 @@
     <parent link="base_link"/>
     <child link="camera_link"/>
-    <origin xyz="0.20 0 0.127" rpy="0 0 0"/>
+    <origin xyz="${camera_forward} 0 ${camera_height - wheel_radius}" rpy="0 0 0"/>
   </joint>
   <link name="camera_infra1_optical_frame"/>
@@ -184,6 +215,6 @@
       <param name="channel">0</param>
       <param name="offset">0.0</param>
-      <param name="min_angle">-0.785</param>
-      <param name="max_angle">0.785</param>
+      <param name="min_angle">${-steer_max_angle}</param>
+      <param name="max_angle">${steer_max_angle}</param>
       <param name="min_pulse_us">1000</param>
       <param name="neutral_pulse_us">1500</param>

Commit message: Record measured wheel diameter and ground clearance (#2)
Wheel diameter 4 in gives radius 0.0508 m in the URDF and steering
controller. Ground clearance measured at 1.5 in = 0.038 m replaces the
estimate. Camera height above ground is unchanged at 0.127 m.

Co-Authored-By: Claude Fable 5.1 <noreply@anthropic.com>
Claude-Session: https://claude.ai/code/session_015xtnKLNTCcXYNkdv7Yybut

File: src/RCCar/rc_hardware_control/description/description.urdf.xacro (robot description, xacro)
@@ -3,16 +3,16 @@
   <!-- ============================================================
        Physical dimensions. Every frame below is derived from these.
-       wheel_radius: owner reported the wheel diameter as "just under
-       4 inches" (2026-09-12), taken as 0.098 m. Replace with a caliper
-       measurement when one is made. The same value must be written in
+       wheel_radius: wheel diameter measured at 4 in = 0.1016 m
+       (2026-09-12). The same value must be written in
        config/steer_bot_hardware.yaml (front/rear_wheel_radius).
-       ground_clearance: ESTIMATE, not yet measured. It only affects
-       where the chassis box is drawn, not any frame, but the obstacle
-       height band in the nvblox config was chosen relative to it.
+       ground_clearance: measured at 1.5 in = 0.038 m (2026-09-12).
+       It only affects where the chassis box is drawn, not any frame,
+       but the obstacle height band in the nvblox config must not start
+       above it or a rock that clears the band will hit the chassis.
        steer_max_angle: the PCA9685 calibration range, not a measured
        mechanical lock. See the turning-radius note in
        config/my_custom_nav2_params.yaml.
        ============================================================ -->
-  <xacro:property name="wheel_radius"      value="0.049"/>
+  <xacro:property name="wheel_radius"      value="0.0508"/>
   <xacro:property name="wheel_width"       value="0.04"/>
   <xacro:property name="wheelbase"         value="0.29"/>
@@ -21,5 +21,5 @@
   <xacro:property name="chassis_width"     value="0.27"/>
   <xacro:property name="chassis_height"    value="0.15"/>
-  <xacro:property name="ground_clearance"  value="0.04"/>   <!-- ESTIMATE: measure -->
+  <xacro:property name="ground_clearance"  value="0.038"/>
   <xacro:property name="camera_height"     value="0.127"/>  <!-- lens centre above ground -->
   <xacro:property name="camera_forward"    value="0.20"/>   <!-- lens ahead of the axle midpoint -->

Commit message: Record measured turning circle and derive the steering lock (#2)
Inside diameter of the minimum turning circle measured at 25 in
(0.635 m) at the inner rear tyre. Rear-axle midpoint radius is therefore
0.45 m and the mechanical lock atan(0.29 / 0.4475) = 0.575 rad (33 deg).

steer_max_angle drops from 0.785 (the PWM calibration range) to 0.575.
The PCA9685 interface maps the angle range linearly onto the pulse range,
so this makes a commanded angle in radians equal the real wheel angle;
previously full lock was reached only at a 0.785 rad command and every
intermediate command under-steered by about 27 percent.

Planner derivation comment updated: the physical floor for base_footprint,
midway between the axles, is 0.47 m. minimum_turning_radius stays at 0.80.

Co-Authored-By: Claude Fable 5.1 <noreply@anthropic.com>
Claude-Session: https://claude.ai/code/session_01JLf9uQcGAfuf7YLT8MgUFQ

File: src/RCCar/rc_hardware_control/description/description.urdf.xacro (robot description, xacro)
@@ -10,7 +10,16 @@
        but the obstacle height band in the nvblox config must not start
        above it or a rock that clears the band will hit the chassis.
-       steer_max_angle: the PCA9685 calibration range, not a measured
-       mechanical lock. See the turning-radius note in
-       config/my_custom_nav2_params.yaml.
+       steer_max_angle: mechanical lock derived from the measured turning
+       circle (2026-09-12): inside diameter 25 in = 0.635 m, taken as the
+       path of the inner rear tyre's inner edge, so the rear-axle midpoint
+       turns at 0.3175 + track_width/2 + wheel_width/2 = 0.4475 m and
+       lock = atan(wheelbase / 0.4475) = 0.575 rad (33 deg). The PCA9685
+       interface maps [-max_angle, max_angle] linearly onto
+       [min_pulse_us, max_pulse_us], so this value is what makes a commanded
+       angle in radians equal the real wheel angle; it assumes a symmetric,
+       linear linkage between the pulse endpoints. If the circle was
+       measured at the tyre centre instead, lock is 0.596 rad; the
+       difference is within measurement error. See the turning-radius note
+       in config/my_custom_nav2_params.yaml.
        ============================================================ -->
   <xacro:property name="wheel_radius"      value="0.0508"/>
@@ -24,5 +33,5 @@
   <xacro:property name="camera_height"     value="0.127"/>  <!-- lens centre above ground -->
   <xacro:property name="camera_forward"    value="0.20"/>   <!-- lens ahead of the axle midpoint -->
-  <xacro:property name="steer_max_angle"   value="0.785"/>  <!-- servo hardware limit, rad -->
+  <xacro:property name="steer_max_angle"   value="0.575"/>  <!-- measured mechanical lock, rad; see header -->
   <!-- Frames:
        base_footprint  ground-contact frame, z = 0 on the floor, midway between the axles.
